Commit message: Add the tf from kinect_link to kinect_depth_optical_frame

File: pedsim_simulator/urdf/p3atstevens.urdf (robot description, URDF)
Before this commit: robot pioneer3at, 25 links, 24 joints
Links:
- added link camera_depth_optical_frame
Joints:
- added joint camera_depth_joint: type fixed, parent kinect_link, child camera_depth_optical_frame, origin xyz=0 0 0 rpy=-1.57 0 -1.57
- joint kinect_joint: axis  -> (none)
